File: emulation4l.kicad_pcb (KiCad board)
At the start: 4 copper layers, 58.4 x 45.1 mm, 94 parts, among them J1 USB_B_Micro, J17 Conn_01x02, J18 Conn_01x02, J19 Conn_01x02, J2 Conn_02x05_Odd_Even, J20 Conn_01x02, J21 Conn_01x02, J22 Conn_02x05_Odd_Even, J4 Conn_02x05_Odd_Even, J5 Conn_01x03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

Commit message: Fixes for Aisler
Parts:
- added FID1: Fiducial, Fiducial:Fiducial_0.5mm_Mask1mm, F.Cu at (167.8, 72.3)
- added FID2: Fiducial, Fiducial:Fiducial_0.5mm_Mask1mm, F.Cu at (167.8, 105.9)
- added FID3: Fiducial, Fiducial:Fiducial_0.5mm_Mask1mm, F.Cu at (114.6, 71.8)
- R29, R32: footprint Resistor_SMD:R_0603_1608Metric -> Resistor_SMD:R_0402_1005Metric
- renumbered J2 to J3
Connections:
- J3 pad 10: (no net) -> /CC_nRESET
- J5 pad 1: /CC_JTAG_nRESET -> (no net)
- J8 pad 10: /CC_JTAG_nRESET -> /CC_nRESET
Routing:
- net /CC_JTAG_nRESET: track 27.2 -> 0.00 mm, vias 1 -> 0
- net /CC_nRESET: track 0.00 -> 24.0 mm, vias 0 -> 1
- net /VCC_BRD: track 63.3 -> 64.0 mm
Other:
- rule pad_to_mask_clearance: 0.051 -> 0.05
- rule solder_mask_min_width: 0.25 -> 0.2
