File: emulation4l.sch (KiCad schematic (older format))
At the start: 90 parts, among them J1 USB_B_Micro, J17 Conn_01x02, J18 Conn_01x02, J19 Conn_01x02, J2 Conn_02x05_Odd_Even, J20 Conn_01x02, J21 Conn_01x02, J22 Conn_02x05_Odd_Even, J4 Conn_02x05_Odd_Even, J5 Conn_01x03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

Commit message: Fixes for Aisler
Parts:
- added FID1, FID2, FID3: Fiducial, Fiducial:Fiducial_0.5mm_Mask1mm, symbol Mechanical:Fiducial
- C1, C14, C17, C24, C25, C4, C5: MFG Name (none) -> TDK; MFG Part Num (none) -> C1005X5R1A104K050BA
- C10, C11, C19: MFG Name (none) -> AVX; MFG Part Num (none) -> 06033D104KAT2A
- C12, C16, C20, C22, C23: MFG Name (none) -> TDK; MFG Part Num (none) -> C1005X5R1C105K050BC
- C13, C6: MFG Name (none) -> Murata; MFG Part Num (none) -> GRM1555C1H220FA01D
- C15, C2, C21, C3, C7, C8, C9: MFG Name (none) -> TDK; MFG Part Num (none) -> C1005X7R1C103K
- C18: MFG Name (none) -> TDK; MFG Part Num (none) -> C1005X5R1C225K050BC
- C60, C62: MFG Name (none) -> Murata; MFG Part Num (none) -> GRM21BR61A106KE19L
- C61: MFG Name (none) -> TDK; MFG Part Num (none) -> C2012X5R1C226K125AC
- D1: MFG Name (none) -> Lumex; MFG Part Num (none) -> SML-LX0603GW-TR
- D2: MFG Name (none) -> Rohm; MFG Part Num (none) -> SML-311UTT86
- D3: MFG Name (none) -> Wurth Elektronik eiSos; MFG Part Num (none) -> 150060YS75000
- FB1, FB2: MFG Name (none) -> Murata; MFG Part Num (none) -> BLM15AG100SN1D
- J1: MFG Name (none) -> Molex; MFG Part Num (none) -> 105017-0001
- J17, J18, J19, J20, J21: MFG Name (none) -> Wurth Elektronik; MFG Part Num (none) -> 61300211121
- J22, J5, J6: MFG Name (none) -> Wurth Elektronik; MFG Part Num (none) -> 61300311121
- J4: MFG Name (none) -> Samtec; MFG Part Num (none) -> FTSH-105-01-F-D-K
- L8: MFG Name (none) -> Taiyo Yuden; MFG Part Num (none) -> BRC2012T2R2MD
- Q1: MFG Name (none) -> Fairchild; MFG Part Num (none) -> BSS138
- R1, R2, R27, R3, R31, R4, R5, R6, R8: MFG Name (none) -> Panasonic; MFG Part Num (none) -> ERJ-2RKF33R0X
- R10, R11, R25, R7, R9: MFG Name (none) -> Vishay-Dale; MFG Part Num (none) -> CRCW04021K00JNED
- R12: MFG Name (none) -> Panasonic; MFG Part Num (none) -> ERJ-2GE0R00X
- R13: MFG Name (none) -> Vishay-Dale; MFG Part Num (none) -> CRCW0402100RJNED
- R14: MFG Name (none) -> Vishay-Dale; MFG Part Num (none) -> CRCW0603100KJNEA
- R145, R24: MFG Name (none) -> Vishay-Dale; MFG Part Num (none) -> CRCW0603270RJNEA
- R146, R17, R26: MFG Name (none) -> Vishay-Dale; MFG Part Num (none) -> CRCW0402100KJNED
- R15: MFG Name (none) -> Vishay-Dale; MFG Part Num (none) -> CRCW0402330KJNED
- R16: MFG Name (none) -> Vishay-Dale; MFG Part Num (none) -> CRCW0402220KJNED
- R18, R19: MFG Name (none) -> Vishay-Dale; MFG Part Num (none) -> CRCW0603220RJNEA
- R20: MFG Name (none) -> Vishay-Dale; MFG Part Num (none) -> CRCW040210K0JNED
- R21: MFG Name (none) -> Panasonic; MFG Part Num (none) -> ERJ-2RKF1000X
- R22: MFG Name (none) -> Vishay-Dale; MFG Part Num (none) -> CRCW0402100RFKED
- R23: MFG Name (none) -> Vishay-Dale; MFG Part Num (none) -> CRCW06034K87FKEA
- R28: MFG Name (none) -> Vishay-Dale; MFG Part Num (none) -> CRCW040251R0JNED
- R29, R32: footprint Resistor_SMD:R_0603_1608Metric -> Resistor_SMD:R_0402_1005Metric; MFG Name (none) -> Vishay-Dale; MFG Part Num (none) -> CRCW04021K00JNED
- SW1: MFG Name (none) -> APEM; MFG Part Num (none) -> MJTP1117
- U1: MFG Name (none) -> Texas Instruments; MFG Part Num (none) -> TM4C1294NCPDTI3R
- U12: MFG Name (none) -> Texas Instruments; MFG Part Num (none) -> TPS62162DSGR
- U2: MFG Name (none) -> Texas Instruments; MFG Part Num (none) -> TPD4S010DQAR
- U3, U4, U6: MFG Name (none) -> Texas Instruments; MFG Part Num (none) -> SN74LVC1T45DCKR
- U5: MFG Name (none) -> Texas Instruments; MFG Part Num (none) -> LM4040B25IDBZR
- Y1: MFG Name (none) -> Abracon; MFG Part Num (none) -> ABM3-16.000MHZ-D2Y-T
- renumbered J2 to J3
Connections:
- net CC_nRESET: now reaches J3.10 (Pin_10)
- net CC_nRESET: now also J8.10 (Pin_10)
- net CC_JTAG_nRESET renamed LP_GPIO_01
- net LP_GPIO_01: no longer J8.10 (Pin_10)
- new net: U1.114 (GND), U1.17 (GND), U1.48 (GND), U1.55 (GND), U1.58 (GND), U1.80 (GND)
